Commit message: Conveyor cell working: RG2 gripper, 0.40m pedestal, config_1 (1->2) + config_2 relay (1->2->3)
Intel-warehouse conveyor cell, both configs verified end-to-end:
- cell_arranged.world: vendored cell_in_warehouse.world with 3 conveyors fanned at
  R~0.82 around the cell + a 0.40m robot_pedestal. UR5 spawned at z=0.40 so the 0.70m
  belts fall inside the floor-arm's top-down reach (IK-verified; floor mount was all UNREACHABLE).
- ur5_rg2_arm.urdf.xacro: RG2 gripper added as COSMETIC visual-only fixed links
  (hand + 2 fingers, mass 1e-4, no collision; transforms/meshes from picknplace ur5_rg2).
- warehouse_pick_place.py: CONFIGS are now conveyor PATHS (config_1=[1,2], config_2=[1,2,3],
  append-only); multi-hop pick/place carries ONE cube along the path (re-picks where the
  previous hop placed it). ROBOT_MOUNT_Z=0.40 (base-frame targets), INWARD=0.27 (near belt
  edge), cube spawns in world frame. Robust arg flattening (launch passes one args string).
- Verified: config_1 places at conv2 within 5mm; config_2 relay re-grasps at conv2 and
  places at conv3 within 2mm. RTF 0.94 with the full warehouse mesh.

File: src/reconfig_cell/cell_bringup/urdf/ur5_rg2_arm.urdf.xacro (robot description, xacro)
@@ -44,4 +44,49 @@
     <origin xyz="0 0 0" rpy="0 0 0"/>
   </xacro:ur_robot>
+  <!-- ── RG2 gripper — COSMETIC visual-only ──────────────────────────────────────
+       The OnRobot RG2 mounted on the flange, so the arm visibly carries its gripper.
+       Fixed links, NEGLIGIBLE mass, and NO <collision>: the grasp is the
+       DetachableJoint (fingers never actuated), and omitting collision keeps the
+       ~0.2 m gripper from jamming into the belt during the flange-level grasp and
+       leaves the verified arm control/planning untouched. Mount + finger transforms
+       and meshes are taken verbatim from picknplace ur5_rg2/model.sdf. -->
+  <xacro:property name="rg2_mesh"
+    value="file://$(env HOME)/picknplace_ws/src/picknplace/urdf/ur5_rg2/meshes/visual/rg2"/>
+  <xacro:macro name="rg2_cosmetic_link" params="name mesh *visual_origin">
+    <link name="${name}">
+      <visual>
+        <xacro:insert_block name="visual_origin"/>
+        <geometry><mesh filename="${rg2_mesh}/${mesh}"/></geometry>
+      </visual>
+      <inertial>
+        <mass value="1e-4"/>
+        <inertia ixx="1e-6" iyy="1e-6" izz="1e-6" ixy="0" ixz="0" iyz="0"/>
+      </inertial>
+    </link>
+  </xacro:macro>
+  <joint name="rg2_hand_joint" type="fixed">
+    <parent link="wrist_3_link"/>
+    <child link="rg2_hand"/>
+    <origin xyz="0 0.0823 0" rpy="1.570796325 0 1.570796325"/>
+  </joint>
+  <xacro:rg2_cosmetic_link name="rg2_hand" mesh="hand.dae">
+    <origin xyz="0 0 0" rpy="0 0 0"/>
+  </xacro:rg2_cosmetic_link>
+  <joint name="rg2_finger_joint1" type="fixed">
+    <parent link="rg2_hand"/>
+    <child link="rg2_leftfinger"/>
+    <origin xyz="0.105 0.017 0" rpy="0 0 0"/>
+  </joint>
+  <xacro:rg2_cosmetic_link name="rg2_leftfinger" mesh="finger.dae">
+    <origin xyz="0 0 0" rpy="0 0 0"/>
+  </xacro:rg2_cosmetic_link>
+  <joint name="rg2_finger_joint2" type="fixed">
+    <parent link="rg2_hand"/>
+    <child link="rg2_rightfinger"/>
+    <origin xyz="0.105 -0.017 0" rpy="0 0 0"/>
+  </joint>
+  <xacro:rg2_cosmetic_link name="rg2_rightfinger" mesh="finger.dae">
+    <origin xyz="0 0 0" rpy="3.141592653589793 0 0"/>
+  </xacro:rg2_cosmetic_link>
   <!-- ros2_control on the 6 arm joints via the stock UR gz macro (position+velocity+effort
        command interfaces; gz_ros2_control needs them to actually drive the joints). The

Commit message: Gripper grabs at fingertips + RG2 mounted flush on the flange
- Grasp TCP moved to the RG2 fingertips (rg2_tcp link) and IK now targets it
  instead of tool0, so the gripper descends vertically with the fingers straddling
  the cube (the wrist's +y gripper axis was pointing the flange-normal grasp
  sideways before). solve_ik + run_diag retargeted to rg2_tcp.
- RG2 visual re-mounted on tool0 (the real flange frame, +z=approach) instead of
  the picknplace wrist_3 frame whose convention differs from stock ur_description --
  the gripper was floating ~8cm off the side, then 8cm out; now flush (xyz 0) with
  fingers along +z. rg2_tcp at 0.193 m (fingertips).
- Robust arg flattening (_tokens) since the launch passes one args:= string.
- Verified: config_1 grasp confirmed, cube placed at conv2 within ~1mm; both
  configs still accurate. User confirmed gripper visually attached + aligned.

File: src/reconfig_cell/cell_bringup/urdf/ur5_rg2_arm.urdf.xacro (robot description, xacro)
@@ -65,8 +65,12 @@
     </link>
   </xacro:macro>
+  <!-- Mounted on tool0 (the real flange frame: +z = approach axis). The picknplace
+       transforms were in ITS wrist_3 frame, which differs from stock ur_description's,
+       so the gripper floated off the side; re-derived here relative to tool0 so the
+       hand sits flush on the flange with the fingers extending along +z. -->
   <joint name="rg2_hand_joint" type="fixed">
-    <parent link="wrist_3_link"/>
+    <parent link="tool0"/>
     <child link="rg2_hand"/>
-    <origin xyz="0 0.0823 0" rpy="1.570796325 0 1.570796325"/>
+    <origin xyz="0 0 0.0" rpy="0 -1.570796327 3.141592654"/>
   </joint>
   <xacro:rg2_cosmetic_link name="rg2_hand" mesh="hand.dae">
@@ -89,4 +93,14 @@
     <origin xyz="0 0 0" rpy="3.141592653589793 0 0"/>
   </xacro:rg2_cosmetic_link>
+  <!-- Grasp TCP at the RG2 fingertips (picknplace ur5_rg2 tool0 transform): this is the
+       frame the IK drives to the belt, so the FINGERS reach the cube instead of the
+       flange. Its +z axis = the wrist's +y = the gripper approach axis, so the existing
+       top-down quaternion (frame +z -> world -z) makes the gripper point straight down. -->
+  <joint name="rg2_tcp_joint" type="fixed">
+    <parent link="tool0"/>
+    <child link="rg2_tcp"/>
+    <origin xyz="0 0 0.193" rpy="0 0 0"/>
+  </joint>
+  <link name="rg2_tcp"/>
   <!-- ros2_control on the 6 arm joints via the stock UR gz macro (position+velocity+effort
        command interfaces; gz_ros2_control needs them to actually drive the joints). The

Commit message: RG2 contact-gated grab: collision fingers that physically clamp the cube
Replace the pure DetachableJoint teleport-weld + cosmetic fingers (box lifted
with a gap, fingers passed through it) with a contact-gated grab: the fingers
must physically close on the cube, then the weld holds it for a stable carry.

urdf/ur5_rg2_arm.urdf.xacro:
- Give rg2_leftfinger/rg2_rightfinger real BOX collision (0.12 0.031 0.02 at
  finger-local 0.047 0 0, mu 1.2) so they stop at the cube instead of through it.
- Widen finger revolute limits to +-1.3 so they can fold fully closed.

scripts/warehouse_pick_place.py:
- Finger sign confirmed visually: POSITIVE = open/spread, NEGATIVE = fold in.
  No tuned grip angle: OPEN=+0.65 to clear the cube, then drive BOTH hard to
  CLOSE=-1.10 and let the cube arrest them (it self-centers between the fingers).
- Fix "only one finger folds": set_fingers() published the gz cmd once per topic
  and a single gz-topic publish is routinely dropped on sim-step timing, leaving
  one finger on its old command. Now publish 4x to both topics so both actuate.

Verified e2e: config_1 (1->2) and config_2 relay (1->2->3, re-pick at conv2)
both grasp-confirm (lift z=0.87) with both fingers clamping at every pick.

File: src/reconfig_cell/cell_bringup/urdf/ur5_rg2_arm.urdf.xacro (robot description, xacro)
@@ -60,6 +60,6 @@
       </visual>
       <inertial>
-        <mass value="1e-4"/>
-        <inertia ixx="1e-6" iyy="1e-6" izz="1e-6" ixy="0" ixz="0" iyz="0"/>
+        <mass value="0.05"/>
+        <inertia ixx="3e-5" iyy="3e-5" izz="3e-5" ixy="0" ixz="0" iyz="0"/>
       </inertial>
     </link>
@@ -77,20 +77,64 @@
     <origin xyz="0 0 0" rpy="0 0 0"/>
   </xacro:rg2_cosmetic_link>
-  <joint name="rg2_finger_joint1" type="fixed">
+  <!-- Fingers are now REVOLUTE so they open/close to pinch the cube. Actuated by gz
+       JointPositionController plugins (below), NOT ros2_control -> decoupled from the
+       verified arm control and avoids the gripper-controller segfault. Driven via gz
+       topics by the demonstrator (open on approach, close on the cube). Axes from
+       picknplace (finger2 mirrored). -->
+  <joint name="rg2_finger_joint1" type="revolute">
     <parent link="rg2_hand"/>
     <child link="rg2_leftfinger"/>
     <origin xyz="0.105 0.017 0" rpy="0 0 0"/>
+    <axis xyz="0 0 1"/>
+    <limit lower="-1.3" upper="1.3" effort="10.6" velocity="1.57"/>
+    <dynamics damping="0.5" friction="0.1"/>
   </joint>
-  <xacro:rg2_cosmetic_link name="rg2_leftfinger" mesh="finger.dae">
-    <origin xyz="0 0 0" rpy="0 0 0"/>
-  </xacro:rg2_cosmetic_link>
-  <joint name="rg2_finger_joint2" type="fixed">
+  <!-- leftfinger: visual mesh + a BOX collision approximating the blade so the
+       finger physically stops at the cube (no more passing through it). Box spans the
+       mesh bounds (local x -0.014..0.108, y ±0.0155, z ±0.010). High friction so the
+       closed fingers actually hold the part by contact. -->
+  <link name="rg2_leftfinger">
+    <visual>
+      <origin xyz="0 0 0" rpy="0 0 0"/>
+      <geometry><mesh filename="${rg2_mesh}/finger.dae"/></geometry>
+    </visual>
+    <collision>
+      <origin xyz="0.047 0 0" rpy="0 0 0"/>
+      <geometry><box size="0.12 0.031 0.02"/></geometry>
+      <surface>
+        <friction><ode><mu>1.2</mu><mu2>1.2</mu2></ode></friction>
+      </surface>
+    </collision>
+    <inertial>
+      <mass value="0.05"/>
+      <inertia ixx="3e-5" iyy="3e-5" izz="3e-5" ixy="0" ixz="0" iyz="0"/>
+    </inertial>
+  </link>
+  <joint name="rg2_finger_joint2" type="revolute">
     <parent link="rg2_hand"/>
     <child link="rg2_rightfinger"/>
     <origin xyz="0.105 -0.017 0" rpy="0 0 0"/>
+    <axis xyz="0 0 -1"/>
+    <limit lower="-1.3" upper="1.3" effort="10.6" velocity="1.57"/>
+    <dynamics damping="0.5" friction="0.1"/>
   </joint>
-  <xacro:rg2_cosmetic_link name="rg2_rightfinger" mesh="finger.dae">
-    <origin xyz="0 0 0" rpy="3.141592653589793 0 0"/>
-  </xacro:rg2_cosmetic_link>
+  <!-- rightfinger: mirror of leftfinger (visual flipped about x), same box collision. -->
+  <link name="rg2_rightfinger">
+    <visual>
+      <origin xyz="0 0 0" rpy="3.141592653589793 0 0"/>
+      <geometry><mesh filename="${rg2_mesh}/finger.dae"/></geometry>
+    </visual>
+    <collision>
+      <origin xyz="0.047 0 0" rpy="0 0 0"/>
+      <geometry><box size="0.12 0.031 0.02"/></geometry>
+      <surface>
+        <friction><ode><mu>1.2</mu><mu2>1.2</mu2></ode></friction>
+      </surface>
+    </collision>
+    <inertial>
+      <mass value="0.05"/>
+      <inertia ixx="3e-5" iyy="3e-5" izz="3e-5" ixy="0" ixz="0" iyz="0"/>
+    </inertial>
+  </link>
   <!-- Grasp TCP at the RG2 fingertips (picknplace ur5_rg2 tool0 transform): this is the
        frame the IK drives to the belt, so the FINGERS reach the cube instead of the
@@ -126,4 +170,21 @@
       <parameters>$(arg simulation_controllers)</parameters>
     </plugin>
+    <!-- RG2 finger position controllers (pure gz, decoupled from ros2_control).
+         Commanded with a gz.msgs.Double target angle on each topic by the
+         demonstrator: open on approach, close on the cube. -->
+    <plugin filename="gz-sim-joint-position-controller-system"
+            name="gz::sim::systems::JointPositionController">
+      <joint_name>rg2_finger_joint1</joint_name>
+      <topic>/rg2/finger1_cmd</topic>
+      <p_gain>8.0</p_gain><i_gain>0.1</i_gain><d_gain>0.4</d_gain>
+      <initial_position>0.0</initial_position>
+    </plugin>
+    <plugin filename="gz-sim-joint-position-controller-system"
+            name="gz::sim::systems::JointPositionController">
+      <joint_name>rg2_finger_joint2</joint_name>
+      <topic>/rg2/finger2_cmd</topic>
+      <p_gain>8.0</p_gain><i_gain>0.1</i_gain><d_gain>0.4</d_gain>
+      <initial_position>0.0</initial_position>
+    </plugin>
   </gazebo>
 </robot>
